Commit message: Fix udrf files

File: realsense_explorer_description/urdf/realsense_bot.urdf (robot description, URDF)
Before this commit: robot realsense_bot, 17 links, 16 joints
Links:
- link rbot_base: mass None -> 0.5
- link servo_bottom: mass None -> 0.2

File: realsense_explorer_description/urdf/realsense_explorer.urdf (robot description, URDF)
Before this commit: robot realsense_explorer, 22 links, 21 joints
Links:
- link U_Link: mass None -> 0.15
- link imu_link: mass None -> 0.000468
- link link_left_wheel: mass None -> 0.456
- link link_right_wheel: mass None -> 0.456
- link rbot_base: mass None -> 0.5
- link robot_base: mass None -> 1.0
- link servo_bottom: mass None -> 0.2
- link servo_mid: mass None -> 0.0477
- link servo_up: mass None -> 0.0477
- link up_mount: mass None -> 0.0999
