Commit message: Add custom targets to update urdf files when xacro updated

File: src/realsense_explorer_description/urdf/realsense_bot.urdf (robot description, URDF)
Before this commit: robot realsense_bot, 17 links, 16 joints
Links:
- link U_Link: mass None -> 0.15
- link servo_mid: mass None -> 0.0477
- link servo_up: mass None -> 0.0477
- link up_mount: mass None -> 0.0999
Joints:
- joint camera_color_optical_joint: origin xyz=0 0 0 rpy=-1.57079632679 0 -1.57079632679 -> xyz=0 0 0 rpy=-1.5707963267948966 0 -1.5707963267948966
- joint camera_depth_optical_joint: origin xyz=0 0 0 rpy=-1.57079632679 0 -1.57079632679 -> xyz=0 0 0 rpy=-1.5707963267948966 0 -1.5707963267948966
- joint camera_infra1_optical_joint: origin xyz=0 0 0 rpy=-1.57079632679 0 -1.57079632679 -> xyz=0 0 0 rpy=-1.5707963267948966 0 -1.5707963267948966
- joint camera_infra2_optical_joint: origin xyz=0 0 0 rpy=-1.57079632679 0 -1.57079632679 -> xyz=0 0 0 rpy=-1.5707963267948966 0 -1.5707963267948966
- joint camera_link_joint: origin xyz=0.0106 0.0175 0.0125 rpy=0 0 0 -> xyz=0.010600000000000002 0.0175 0.0125 rpy=0 0 0

File: src/realsense_explorer_description/urdf/realsense_bot.urdf.xacro (robot description, xacro)
@@ -26,4 +26,9 @@
        <material name="blue"/>
     </visual>
+    <inertial>
+      <mass value="0.5"/>
+      <origin xyz="0 0 0"/>
+      <inertia ixx="0.000375" ixy="0.0" ixz="0.0" iyy="0.000122" iyz="0.0" izz="0.000422"/>
+    </inertial>
   </link>
   <link name="servo_bottom">
@@ -35,4 +40,9 @@
       <material name="red"/>
     </visual>
+    <inertial>
+      <mass value="0.2"/>
+      <origin xyz="0 0 0"/>
+      <inertia ixx="2.5e-05" ixy="0.0" ixz="0.0" iyy="1.25e-05" iyz="0.0" izz="2.5e-05"/>
+    </inertial>
   </link>
   <link name="U_Link">
@@ -44,4 +54,9 @@
       <material name="blue"/>
     </visual>
+    <inertial>
+      <mass value="0.15"/>
+      <origin xyz="0 0 0"/>
+      <inertia ixx="4.6933e-05" ixy="0.0" ixz="0.0" iyy="1.4062e-05" iyz="0.0" izz="3.6094e-06"/>
+    </inertial>
   </link>
   <link name="servo_mid">
@@ -53,4 +68,9 @@
       <material name="red"/>
     </visual>
+    <inertial>
+      <mass value="0.0477"/>
+      <origin xyz="0 0 0"/>
+      <inertia ixx="4.4887e-06" ixy="0.0" ixz="0.0" iyy="2.2443e-06" iyz="0.0" izz="4.4887e-06"/>
+   </inertial>
   </link>
   <link name="servo_up">
@@ -62,4 +82,9 @@
       <material name="red"/>
     </visual>
+    <inertial>
+      <mass value="0.0477"/>
+      <origin xyz="0 0 0"/>
+      <inertia ixx="4.4887e-06" ixy="0.0" ixz="0.0" iyy="2.2443e-06" iyz="0.0" izz="4.4887e-06"/>
+    </inertial>
   </link>
   <link name="up_mount">
@@ -71,4 +96,9 @@
       <material name="white"/>
     </visual>
+    <inertial>
+      <mass value="0.0999"/>
+      <origin xyz="0 0 0"/>
+      <inertia ixx="9.2267e-05" ixy="0.0" ixz="0.0" iyy="1.8252e-05" iyz="0.0" izz="9.2267e-05"/>
+    </inertial>
   </link>
   <joint name="base_to_Servo_B" type="fixed">

File: src/realsense_explorer_description/urdf/realsense_explorer.urdf (robot description, URDF)
Before this commit: robot realsense_explorer, 22 links, 21 joints
Joints:
- joint camera_color_optical_joint: origin xyz=0 0 0 rpy=-1.57079632679 0 -1.57079632679 -> xyz=0 0 0 rpy=-1.5707963267948966 0 -1.5707963267948966
- joint camera_depth_optical_joint: origin xyz=0 0 0 rpy=-1.57079632679 0 -1.57079632679 -> xyz=0 0 0 rpy=-1.5707963267948966 0 -1.5707963267948966
- joint camera_infra1_optical_joint: origin xyz=0 0 0 rpy=-1.57079632679 0 -1.57079632679 -> xyz=0 0 0 rpy=-1.5707963267948966 0 -1.5707963267948966
- joint camera_infra2_optical_joint: origin xyz=0 0 0 rpy=-1.57079632679 0 -1.57079632679 -> xyz=0 0 0 rpy=-1.5707963267948966 0 -1.5707963267948966
- joint camera_link_joint: origin xyz=0.0106 0.0175 0.0125 rpy=0 0 0 -> xyz=0.010600000000000002 0.0175 0.0125 rpy=0 0 0

File: src/realsense_explorer_description/urdf/realsense_explorer.urdf.xacro (robot description, xacro)
@@ -29,4 +29,10 @@
       </geometry>
     </collision>
+    <inertial>
+      <mass value="1.0"/>
+      <origin xyz="0 0 0"/>
+      <inertia ixx="0.0167" ixy="0.0" ixz="0.0"
+           iyy="0.0208" iyz="0.0" izz="0.0108"/>
+    </inertial>
   </link>
     <joint name="base_joint" type="fixed">
@@ -54,4 +60,10 @@
     <material name="invisible"/>
   </visual>
+  <inertial>
+    <mass value="0.456"/>
+    <origin xyz="0 0 0"/>
+    <inertia ixx="0.000766" ixy="0.0" ixz="0.0"
+           iyy="0.000766" iyz="0.0" izz="0.000686"/>
+  </inertial>
 </link>
 <joint name="joint_right_wheel" type="continuous">
@@ -77,4 +89,10 @@
     <material name="invisible"/>
   </visual>
+  <inertial>
+    <mass value="0.456"/>
+    <origin xyz="0 0 0"/>
+    <inertia ixx="0.000766" ixy="0.0" ixz="0.0"
+           iyy="0.000766" iyz="0.0" izz="0.000686"/>
+  </inertial>
 </link>
 <joint name="joint_left_wheel" type="continuous">
@@ -86,5 +104,5 @@
   <joint_properties damping="1.0" friction="1.0" />
 </joint>
-  <link name="imu_link">
+<link name="imu_link">
     <visual>
       <geometry>
@@ -93,5 +111,11 @@
       <material name="green"/>
     </visual>
-  </link>
+    <inertial>
+      <mass value="0.000468"/>
+      <origin xyz="0 0 0"/>
+      <inertia ixx="1.4e-7" ixy="0.0" ixz="0.0"
+           iyy="4.3e-7" iyz="0.0" izz="6.1e-7"/>
+    </inertial>
+</link>
 <joint name="imu_joint" type="fixed">
   <origin rpy="0 0 0" xyz="0.114 0 0.05"/>
