Commit message: Move camera in front of robot withot servo

File: src/realsense_explorer_description/urdf/realsense_explorer.urdf (robot description, URDF)
Before this commit: robot realsense_explorer, 22 links, 21 joints
Links:
- removed link U_Link
- removed link rbot_base
- removed link servo_bottom
- removed link servo_mid
- removed link servo_up
- removed link up_mount
Joints:
- removed joint Joint_1
- removed joint Joint_2
- removed joint Joint_3
- removed joint base_to_Servo_B
- removed joint mount_to_camera
- removed joint servo_mid_to_servo_up
- joint camera_joint: origin xyz=0 0 0 rpy=0 0 0 -> xyz=0.08 0 -0.035 rpy=0 0 0
- joint chasis_to_rbot: child rbot_base -> base_link; origin xyz=-0.09 0 0.13787 rpy=0 0 0 -> xyz=0 0 0.125 rpy=0 0 0

File: src/realsense_explorer_description/urdf/realsense_explorer.urdf.xacro (robot description, xacro)
@@ -4,5 +4,9 @@
   <xacro:arg name="add_plug" default="false" />
   <xacro:arg name="use_mesh" default="true" />
-  <xacro:include filename="$(find realsense_explorer_description)/urdf/realsense_bot.urdf.xacro" />
+  <xacro:include filename="$(find realsense2_description)/urdf/_d435.urdf.xacro" />
+  <link name="base_link" />
+  <xacro:sensor_d435 parent="base_link" use_nominal_extrinsics="true" add_plug="false" use_mesh="true">
+    <origin xyz="0.08 0 -0.035" rpy="0 0 0"/>
+  </xacro:sensor_d435>
   <material name="invisible">
     <color rgba="0 0 0 0"/>
@@ -43,6 +47,6 @@
   <joint name="chasis_to_rbot" type="fixed">
     <parent link="robot_base"/>
-    <child link="rbot_base"/>
-    <origin xyz="-0.09 0 0.13787" rpy="0 0 0"/>
+    <child link="base_link"/>
+    <origin xyz="0 0 0.125" rpy="0 0 0"/>
   </joint>
 <link name="link_right_wheel">

Commit message: Add realsense plugin to gazebo to view camera in rviz and use pointcloud

File: src/realsense_explorer_description/urdf/realsense_explorer.urdf (robot description, URDF)
Before this commit: robot realsense_explorer, 16 links, 15 joints
Links:
- removed link camera_infra1_frame
- removed link camera_infra1_optical_frame
- removed link camera_infra2_frame
- removed link camera_infra2_optical_frame
- added link camera_left_ir_frame
- added link camera_left_ir_optical_frame
- added link camera_right_ir_frame
- added link camera_right_ir_optical_frame
- link camera_link: mass 0.072 -> 0.564
Joints:
- removed joint camera_infra1_joint
- removed joint camera_infra1_optical_joint
- removed joint camera_infra2_joint
- removed joint camera_infra2_optical_joint
- added joint camera_left_ir_joint: type fixed, parent camera_depth_frame, child camera_left_ir_frame, origin xyz=0 0.0 0 rpy=0 0 0
- added joint camera_left_ir_optical_joint: type fixed, parent camera_left_ir_frame, child camera_left_ir_optical_frame, origin xyz=0 0 0 rpy=-1.5707963267948966 0 -1.5707963267948966
- added joint camera_right_ir_joint: type fixed, parent camera_depth_frame, child camera_right_ir_frame, origin xyz=0 -0.05 0 rpy=0 0 0
- added joint camera_right_ir_optical_joint: type fixed, parent camera_right_ir_frame, child camera_right_ir_optical_frame, origin xyz=0 0 0 rpy=-1.5707963267948966 0 -1.5707963267948966
- joint camera_color_joint: parent camera_link -> camera_depth_frame
- joint camera_link_joint: origin xyz=0.010600000000000002 0.0175 0.0125 rpy=0 0 0 -> xyz=0 0.0175 0.0125 rpy=0 0 0

File: src/realsense_explorer_description/urdf/realsense_explorer.urdf.xacro (robot description, xacro)
@@ -1,11 +1,8 @@
 <?xml version="1.0"?>
 <robot xmlns:xacro="http://www.ros.org/wiki/xacro" name="realsense_explorer">
-  <xacro:arg name="use_nominal_extrinsics" default="false"/>
-  <xacro:arg name="add_plug" default="false" />
-  <xacro:arg name="use_mesh" default="true" />
   <xacro:include filename="$(find realsense2_description)/urdf/_d435.urdf.xacro" />
   <link name="base_link" />
-  <xacro:sensor_d435 parent="base_link" use_nominal_extrinsics="true" add_plug="false" use_mesh="true">
-    <origin xyz="0.08 0 -0.035" rpy="0 0 0"/>
+  <xacro:sensor_d435 name="camera" topics_ns="camera" parent="base_link" publish_pointcloud="true">
+    <origin xyz="0.08 0 -0.035" rpy="0 0 0" />
   </xacro:sensor_d435>
   <material name="invisible">
@@ -18,5 +15,5 @@
     <color rgba="0.9 0.9 0.9 1"/>
   </material>
-<link name="base_footprint"/>
+  <link name="base_footprint"/>
   <link name="robot_base">
     <visual>
@@ -27,5 +24,5 @@
       <material name="grey"/>
     </visual>
-      <collision>
+    <collision>
       <origin rpy="1.57 0 3.14" xyz="0.15 -0.117 0"/>
       <geometry>
@@ -40,9 +37,9 @@
     </inertial>
   </link>
-    <joint name="base_joint" type="fixed">
-      <origin rpy="0 0 0" xyz="0 0 0" />
-      <parent link="base_footprint"/>
-      <child link="robot_base" />
-    </joint>
+  <joint name="base_joint" type="fixed">
+    <origin rpy="0 0 0" xyz="0 0 0" />
+    <parent link="base_footprint"/>
+    <child link="robot_base" />
+  </joint>
   <joint name="chasis_to_rbot" type="fixed">
     <parent link="robot_base"/>
@@ -50,108 +47,108 @@
     <origin xyz="0 0 0.125" rpy="0 0 0"/>
   </joint>
-<link name="link_right_wheel">
-  <collision name="link_right_wheel_visual">
-    <origin rpy="0 1.5707 1.57" xyz="0 0 0"/>
-    <geometry>
-      <cylinder length="0.04" radius="0.055"/>
-    </geometry>
-  </collision>
-  <visual name="link_right_wheel_visual">
-    <origin rpy="0 1.5707 1.57" xyz="0 0 0"/>
-    <geometry>
-      <cylinder length="0.04" radius="0.055"/>
-    </geometry>
-    <material name="invisible"/>
-  </visual>
-  <inertial>
-    <mass value="0.456"/>
-    <origin xyz="0 0 0"/>
-    <inertia ixx="0.000766" ixy="0.0" ixz="0.0"
-           iyy="0.000766" iyz="0.0" izz="0.000686"/>
-  </inertial>
-</link>
-<joint name="joint_right_wheel" type="continuous">
-  <origin rpy="0 0 0" xyz="0 -0.1 0.055"/>
-  <child link="link_right_wheel" />
-  <parent link="robot_base"/>
-  <axis rpy="0 0 0" xyz="0 1 0"/>
-  <limit effort="10000" velocity="1000"/>
-  <joint_properties damping="1.0" friction="1.0" />
-</joint>
-<link name="link_left_wheel">
-  <collision name="link_left_wheel_visual">
-    <origin rpy="0 1.5707 1.57" xyz="0 0 0"/>
-    <geometry>
-      <cylinder length="0.04" radius="0.055"/>
-    </geometry>
-  </collision>
-  <visual name="link_left_wheel_visual">
-    <origin rpy="0 1.5707 1.57" xyz="0 0 0"/>
-    <geometry>
-      <cylinder length="0.04" radius="0.055"/>
-    </geometry>
-    <material name="invisible"/>
-  </visual>
-  <inertial>
-    <mass value="0.456"/>
-    <origin xyz="0 0 0"/>
-    <inertia ixx="0.000766" ixy="0.0" ixz="0.0"
-           iyy="0.000766" iyz="0.0" izz="0.000686"/>
-  </inertial>
-</link>
-<joint name="joint_left_wheel" type="continuous">
-  <origin rpy="0 0 0" xyz="0 0.1 0.055"/>
-  <child link="link_left_wheel" />
-  <parent link="robot_base"/>
-  <axis rpy="0 0 0" xyz="0 1 0"/>
-  <limit effort="10000" velocity="1000"/>
-  <joint_properties damping="1.0" friction="1.0" />
-</joint>
-<link name="imu_link">
-    <visual>
+  <link name="link_right_wheel">
+    <collision name="link_right_wheel_visual">
+      <origin rpy="0 1.5707 1.57" xyz="0 0 0"/>
       <geometry>
-        <box size="0.015 0.026 0.001"/>
+        <cylinder length="0.04" radius="0.055"/>
       </geometry>
-      <material name="green"/>
+    </collision>
+    <visual name="link_right_wheel_visual">
+      <origin rpy="0 1.5707 1.57" xyz="0 0 0"/>
+      <geometry>
+        <cylinder length="0.04" radius="0.055"/>
+      </geometry>
+      <material name="invisible"/>
     </visual>
     <inertial>
-      <mass value="0.000468"/>
+      <mass value="0.456"/>
       <origin xyz="0 0 0"/>
-      <inertia ixx="1.4e-7" ixy="0.0" ixz="0.0"
-           iyy="4.3e-7" iyz="0.0" izz="6.1e-7"/>
+      <inertia ixx="0.000766" ixy="0.0" ixz="0.0"
+             iyy="0.000766" iyz="0.0" izz="0.000686"/>
     </inertial>
-</link>
-<joint name="imu_joint" type="fixed">
-  <origin rpy="0 0 0" xyz="0.114 0 0.05"/>
-  <child link="imu_link" />
-  <parent link="robot_base"/>
-</joint>
-<transmission name="right_wheel_transmission">
-  <type>transmission_interface/SimpleTransmission</type>
-  <joint name="joint_right_wheel">
-    <hardwareInterface>
-      hardware_interface/VelocityJointInterface
-    </hardwareInterface>
+  </link>
+  <joint name="joint_right_wheel" type="continuous">
+    <origin rpy="0 0 0" xyz="0 -0.1 0.055"/>
+    <child link="link_right_wheel" />
+    <parent link="robot_base"/>
+    <axis rpy="0 0 0" xyz="0 1 0"/>
+    <limit effort="10000" velocity="1000"/>
+    <joint_properties damping="1.0" friction="1.0" />
   </joint>
-  <actuator name="right_wheel_actuator">
-    <mechanicalReduction>1</mechanicalReduction>
-    <hardwareInterface>
-      VelocityJointInterface
-    </hardwareInterface>
-  </actuator>
-</transmission>
-<transmission name="left_wheel_transmission">
-  <type>transmission_interface/SimpleTransmission</type>
-  <joint name="joint_left_wheel">
-    <hardwareInterface>
-      hardware_interface/VelocityJointInterface
-    </hardwareInterface>
+  <link name="link_left_wheel">
+    <collision name="link_left_wheel_visual">
+      <origin rpy="0 1.5707 1.57" xyz="0 0 0"/>
+      <geometry>
+        <cylinder length="0.04" radius="0.055"/>
+      </geometry>
+    </collision>
+    <visual name="link_left_wheel_visual">
+      <origin rpy="0 1.5707 1.57" xyz="0 0 0"/>
+      <geometry>
+        <cylinder length="0.04" radius="0.055"/>
+      </geometry>
+      <material name="invisible"/>
+    </visual>
+    <inertial>
+      <mass value="0.456"/>
+      <origin xyz="0 0 0"/>
+      <inertia ixx="0.000766" ixy="0.0" ixz="0.0"
+             iyy="0.000766" iyz="0.0" izz="0.000686"/>
+    </inertial>
+  </link>
+  <joint name="joint_left_wheel" type="continuous">
+    <origin rpy="0 0 0" xyz="0 0.1 0.055"/>
+    <child link="link_left_wheel" />
+    <parent link="robot_base"/>
+    <axis rpy="0 0 0" xyz="0 1 0"/>
+    <limit effort="10000" velocity="1000"/>
+    <joint_properties damping="1.0" friction="1.0" />
   </joint>
-  <actuator name="left_wheel_actuator">
-    <mechanicalReduction>1</mechanicalReduction>
-    <hardwareInterface>
-      VelocityJointInterface
-    </hardwareInterface>
-  </actuator>
-</transmission>
+  <link name="imu_link">
+      <visual>
+        <geometry>
+          <box size="0.015 0.026 0.001"/>
+        </geometry>
+        <material name="green"/>
+      </visual>
+      <inertial>
+        <mass value="0.000468"/>
+        <origin xyz="0 0 0"/>
+        <inertia ixx="1.4e-7" ixy="0.0" ixz="0.0"
+             iyy="4.3e-7" iyz="0.0" izz="6.1e-7"/>
+      </inertial>
+  </link>
+  <joint name="imu_joint" type="fixed">
+    <origin rpy="0 0 0" xyz="0.114 0 0.05"/>
+    <child link="imu_link" />
+    <parent link="robot_base"/>
+  </joint>
+  <transmission name="right_wheel_transmission">
+    <type>transmission_interface/SimpleTransmission</type>
+    <joint name="joint_right_wheel">
+      <hardwareInterface>
+        hardware_interface/VelocityJointInterface
+      </hardwareInterface>
+    </joint>
+    <actuator name="right_wheel_actuator">
+      <mechanicalReduction>1</mechanicalReduction>
+      <hardwareInterface>
+        VelocityJointInterface
+      </hardwareInterface>
+    </actuator>
+  </transmission>
+  <transmission name="left_wheel_transmission">
+    <type>transmission_interface/SimpleTransmission</type>
+    <joint name="joint_left_wheel">
+      <hardwareInterface>
+        hardware_interface/VelocityJointInterface
+      </hardwareInterface>
+    </joint>
+    <actuator name="left_wheel_actuator">
+      <mechanicalReduction>1</mechanicalReduction>
+      <hardwareInterface>
+        VelocityJointInterface
+      </hardwareInterface>
+    </actuator>
+  </transmission>
 </robot>

Commit message: Enable diff drive

File: src/realsense_explorer_description/urdf/realsense_explorer.urdf (robot description, URDF)
Before this commit: robot realsense_explorer, 16 links, 15 joints
Joints:
- joint joint_left_wheel: limit effort=10000 velocity=1000 -> effort=100 velocity=10
- joint joint_right_wheel: limit effort=10000 velocity=1000 -> effort=100 velocity=10

File: src/realsense_explorer_description/urdf/realsense_explorer.urdf.xacro (robot description, xacro)
@@ -15,4 +15,7 @@
     <color rgba="0.9 0.9 0.9 1"/>
   </material>
+  <gazebo>
+    <plugin name="gazebo_ros_control" filename="libgazebo_ros_control.so"/>
+  </gazebo>
   <link name="base_footprint"/>
   <link name="robot_base">
@@ -59,5 +62,5 @@
         <cylinder length="0.04" radius="0.055"/>
       </geometry>
-      <material name="invisible"/>
+      <material name="green"/>
     </visual>
     <inertial>
@@ -72,6 +75,6 @@
     <child link="link_right_wheel" />
     <parent link="robot_base"/>
-    <axis rpy="0 0 0" xyz="0 1 0"/>
-    <limit effort="10000" velocity="1000"/>
+    <axis xyz="0 1 0"/>
+    <limit effort="100" velocity="10"/>
     <joint_properties damping="1.0" friction="1.0" />
   </joint>
@@ -88,5 +91,5 @@
         <cylinder length="0.04" radius="0.055"/>
       </geometry>
-      <material name="invisible"/>
+      <material name="green"/>
     </visual>
     <inertial>
@@ -101,6 +104,6 @@
     <child link="link_left_wheel" />
     <parent link="robot_base"/>
-    <axis rpy="0 0 0" xyz="0 1 0"/>
-    <limit effort="10000" velocity="1000"/>
+    <axis xyz="0 1 0"/>
+    <limit effort="100" velocity="10"/>
     <joint_properties damping="1.0" friction="1.0" />
   </joint>
