Commit message: Add skid steering drive to gazebo simulation

File: src/realsense_explorer_description/urdf/realsense_explorer.urdf (robot description, URDF)
Before this commit: robot realsense_explorer, 16 links, 15 joints
Links:
- removed link link_left_wheel
- removed link link_right_wheel
- added link link_back_left_wheel, mass 0.456; collision cylinder length=0.02 radius=0.02; visual cylinder length=0.02 radius=0.02
- added link link_back_right_wheel, mass 0.456; collision cylinder length=0.02 radius=0.02; visual cylinder length=0.02 radius=0.02
- added link link_front_left_wheel, mass 0.456; collision cylinder length=0.02 radius=0.02; visual cylinder length=0.02 radius=0.02
- added link link_front_right_wheel, mass 0.456; collision cylinder length=0.02 radius=0.02; visual cylinder length=0.02 radius=0.02
Joints:
- removed joint joint_left_wheel
- removed joint joint_right_wheel
- added joint joint_back_left_wheel: type continuous, parent robot_base, child link_back_left_wheel, origin xyz=-0.073 0.08 0.02 rpy=0 0 0, axis 0 1 0, limit effort=100 velocity=10
- added joint joint_back_right_wheel: type continuous, parent robot_base, child link_back_right_wheel, origin xyz=-0.073 -0.08 0.02 rpy=0 0 0, axis 0 1 0, limit effort=100 velocity=10
- added joint joint_front_left_wheel: type continuous, parent robot_base, child link_front_left_wheel, origin xyz=0.095 0.08 0.02 rpy=0 0 0, axis 0 1 0, limit effort=100 velocity=10
- added joint joint_front_right_wheel: type continuous, parent robot_base, child link_front_right_wheel, origin xyz=0.095 -0.08 0.02 rpy=0 0 0, axis 0 1 0, limit effort=100 velocity=10
- joint base_joint: child robot_base -> base_link
- joint camera_joint: origin xyz=0.08 0 -0.035 rpy=0 0 0 -> xyz=0.08 0 0.09 rpy=0 0 0; parent base_link -> robot_base
- joint chasis_to_rbot: child base_link -> robot_base; origin xyz=0 0 0.125 rpy=0 0 0 -> xyz=0 0 0 rpy=0 0 0; parent robot_base -> base_link

File: src/realsense_explorer_description/urdf/realsense_explorer.urdf.xacro (robot description, xacro)
@@ -3,6 +3,6 @@
   <xacro:include filename="$(find realsense2_description)/urdf/_d435.urdf.xacro" />
   <link name="base_link" />
-  <xacro:sensor_d435 name="camera" topics_ns="camera" parent="base_link" publish_pointcloud="true">
-    <origin xyz="0.08 0 -0.035" rpy="0 0 0" />
+  <xacro:sensor_d435 name="camera" topics_ns="camera" parent="robot_base" publish_pointcloud="true">
+    <origin xyz="0.08 0 0.09" rpy="0 0 0" />
   </xacro:sensor_d435>
   <material name="invisible">
@@ -16,5 +16,25 @@
   </material>
   <gazebo>
-    <plugin name="gazebo_ros_control" filename="libgazebo_ros_control.so"/>
+    <plugin name="skid_steer_drive_controller" filename="libgazebo_ros_skid_steer_drive.so">
+      <updateRate>100.0</updateRate>
+      <robotNamespace>/</robotNamespace>
+      <leftFrontJoint>joint_front_left_wheel</leftFrontJoint>
+      <rightFrontJoint>joint_front_right_wheel</rightFrontJoint>
+      <leftRearJoint>joint_back_left_wheel</leftRearJoint>
+      <rightRearJoint>joint_back_right_wheel</rightRearJoint>
+      <wheelSeparation>0.2</wheelSeparation>
+      <wheelDiameter>0.2</wheelDiameter>
+      <robotBaseFrame>base_footprint</robotBaseFrame>
+      <torque>20</torque>
+      <maxVelocity>2.0</maxVelocity>
+      <maxAcceleration>3.0</maxAcceleration>
+      <topicName>cmd_vel</topicName>
+      <odometryTopic>odom</odometryTopic>
+      <odometryFrame>odom</odometryFrame>
+      <broadcastTF>true</broadcastTF>
+      <covariance_x>0.0001</covariance_x>
+      <covariance_y>0.0001</covariance_y>
+      <covariance_yaw>0.01</covariance_yaw>
+    </plugin>
   </gazebo>
   <link name="base_footprint"/>
@@ -43,69 +63,132 @@
     <origin rpy="0 0 0" xyz="0 0 0" />
     <parent link="base_footprint"/>
-    <child link="robot_base" />
+    <child link="base_link" />
   </joint>
   <joint name="chasis_to_rbot" type="fixed">
-    <parent link="robot_base"/>
-    <child link="base_link"/>
-    <origin xyz="0 0 0.125" rpy="0 0 0"/>
-  </joint>
-  <link name="link_right_wheel">
-    <collision name="link_right_wheel_visual">
-      <origin rpy="0 1.5707 1.57" xyz="0 0 0"/>
-      <geometry>
-        <cylinder length="0.04" radius="0.055"/>
-      </geometry>
-    </collision>
-    <visual name="link_right_wheel_visual">
-      <origin rpy="0 1.5707 1.57" xyz="0 0 0"/>
-      <geometry>
-        <cylinder length="0.04" radius="0.055"/>
-      </geometry>
-      <material name="green"/>
-    </visual>
-    <inertial>
-      <mass value="0.456"/>
-      <origin xyz="0 0 0"/>
-      <inertia ixx="0.000766" ixy="0.0" ixz="0.0"
-             iyy="0.000766" iyz="0.0" izz="0.000686"/>
-    </inertial>
-  </link>
-  <joint name="joint_right_wheel" type="continuous">
-    <origin rpy="0 0 0" xyz="0 -0.1 0.055"/>
-    <child link="link_right_wheel" />
-    <parent link="robot_base"/>
-    <axis xyz="0 1 0"/>
-    <limit effort="100" velocity="10"/>
-    <joint_properties damping="1.0" friction="1.0" />
-  </joint>
-  <link name="link_left_wheel">
-    <collision name="link_left_wheel_visual">
-      <origin rpy="0 1.5707 1.57" xyz="0 0 0"/>
-      <geometry>
-        <cylinder length="0.04" radius="0.055"/>
-      </geometry>
-    </collision>
-    <visual name="link_left_wheel_visual">
-      <origin rpy="0 1.5707 1.57" xyz="0 0 0"/>
-      <geometry>
-        <cylinder length="0.04" radius="0.055"/>
-      </geometry>
-      <material name="green"/>
-    </visual>
-    <inertial>
-      <mass value="0.456"/>
-      <origin xyz="0 0 0"/>
-      <inertia ixx="0.000766" ixy="0.0" ixz="0.0"
-             iyy="0.000766" iyz="0.0" izz="0.000686"/>
-    </inertial>
-  </link>
-  <joint name="joint_left_wheel" type="continuous">
-    <origin rpy="0 0 0" xyz="0 0.1 0.055"/>
-    <child link="link_left_wheel" />
-    <parent link="robot_base"/>
-    <axis xyz="0 1 0"/>
-    <limit effort="100" velocity="10"/>
-    <joint_properties damping="1.0" friction="1.0" />
-  </joint>
+    <parent link="base_link"/>
+    <child link="robot_base"/>
+    <origin xyz="0 0 0" rpy="0 0 0"/>
+  </joint>
+  <!-- Front Right Wheel -->
+  <link name="link_front_right_wheel">
+    <collision name="link_front_right_wheel_visual">
+      <origin rpy="1.5707 0 0" xyz="0 0 0"/>
+      <geometry>
+        <cylinder length="0.02" radius="0.02"/>
+      </geometry>
+    </collision>
+    <visual name="link_front_right_wheel_visual">
+      <origin rpy="1.5707 0 0" xyz="0 0 0"/>
+      <geometry>
+        <cylinder length="0.02" radius="0.02"/>
+      </geometry>
+      <material name="green"/>
+    </visual>
+    <inertial>
+      <mass value="0.456"/>
+      <origin xyz="0 0 0"/>
+      <inertia ixx="6.08e-5" ixy="0.0" ixz="0.0"
+           iyy="6.08e-5" iyz="0.0" izz="9.12e-5"/>
+    </inertial>
+  </link>
+  <joint name="joint_front_right_wheel" type="continuous">
+    <origin rpy="0 0 0" xyz="0.095 -0.08 0.02"/>
+    <child link="link_front_right_wheel" />
+    <parent link="robot_base"/>
+    <axis xyz="0 1 0"/>
+    <limit effort="100" velocity="10"/>
+    <joint_properties damping="1.0" friction="1.0" />
+  </joint>
+  <!-- Front Left Wheel -->
+  <link name="link_front_left_wheel">
+    <collision name="link_front_right_wheel_visual">
+      <origin rpy="1.5707 0 0" xyz="0 0 0"/>
+      <geometry>
+        <cylinder length="0.02" radius="0.02"/>
+      </geometry>
+    </collision>
+    <visual name="link_front_right_wheel_visual">
+      <origin rpy="1.5707 0 0" xyz="0 0 0"/>
+      <geometry>
+        <cylinder length="0.02" radius="0.02"/>
+      </geometry>
+      <material name="green"/>
+    </visual>
+    <inertial>
+      <mass value="0.456"/>
+      <origin xyz="0 0 0"/>
+      <inertia ixx="6.08e-5" ixy="0.0" ixz="0.0"
+           iyy="6.08e-5" iyz="0.0" izz="9.12e-5"/>
+    </inertial>
+  </link>
+  <joint name="joint_front_left_wheel" type="continuous">
+    <origin rpy="0 0 0" xyz="0.095 0.08 0.02"/>
+    <child link="link_front_left_wheel" />
+    <parent link="robot_base"/>
+    <axis xyz="0 1 0"/>
+    <limit effort="100" velocity="10"/>
+    <joint_properties damping="1.0" friction="1.0" />
+  </joint>
+  <!-- Back Left Wheel -->
+  <link name="link_back_left_wheel">
+    <collision name="link_back_right_wheel_visual">
+      <origin rpy="1.5707 0 0" xyz="0 0 0"/>
+      <geometry>
+        <cylinder length="0.02" radius="0.02"/>
+      </geometry>
+    </collision>
+    <visual name="link_back_right_wheel_visual">
+      <origin rpy="1.5707 0 0" xyz="0 0 0"/>
+      <geometry>
+        <cylinder length="0.02" radius="0.02"/>
+      </geometry>
+      <material name="green"/>
+    </visual>
+    <inertial>
+      <mass value="0.456"/>
+      <origin xyz="0 0 0"/>
+      <inertia ixx="6.08e-5" ixy="0.0" ixz="0.0"
+           iyy="6.08e-5" iyz="0.0" izz="9.12e-5"/>
+    </inertial>
+  </link>
+  <joint name="joint_back_left_wheel" type="continuous">
+    <origin rpy="0 0 0" xyz="-0.073 0.08 0.02"/>
+    <child link="link_back_left_wheel" />
+    <parent link="robot_base"/>
+    <axis xyz="0 1 0"/>
+    <limit effort="100" velocity="10"/>
+    <joint_properties damping="1.0" friction="1.0" />
+  </joint>
+  <!-- Back Right Wheel -->
+  <link name="link_back_right_wheel">
+    <collision name="link_back_right_wheel_visual">
+      <origin rpy="1.5707 0 0" xyz="0 0 0"/>
+      <geometry>
+        <cylinder length="0.02" radius="0.02"/>
+      </geometry>
+    </collision>
+    <visual name="link_back_right_wheel_visual">
+      <origin rpy="1.5707 0 0" xyz="0 0 0"/>
+      <geometry>
+        <cylinder length="0.02" radius="0.02"/>
+      </geometry>
+      <material name="green"/>
+    </visual>
+    <inertial>
+      <mass value="0.456"/>
+      <origin xyz="0 0 0"/>
+      <inertia ixx="6.08e-5" ixy="0.0" ixz="0.0"
+           iyy="6.08e-5" iyz="0.0" izz="9.12e-5"/>
+    </inertial>
+  </link>
+  <joint name="joint_back_right_wheel" type="continuous">
+    <origin rpy="0 0 0" xyz="-0.073 -0.08 0.02"/>
+    <child link="link_back_right_wheel" />
+    <parent link="robot_base"/>
+    <axis xyz="0 1 0"/>
+    <limit effort="100" velocity="10"/>
+    <joint_properties damping="1.0" friction="1.0" />
+  </joint>
+  <!-- IMU Link -->
   <link name="imu_link">
       <visual>
@@ -127,31 +210,3 @@
     <parent link="robot_base"/>
   </joint>
-  <transmission name="right_wheel_transmission">
-    <type>transmission_interface/SimpleTransmission</type>
-    <joint name="joint_right_wheel">
-      <hardwareInterface>
-        hardware_interface/VelocityJointInterface
-      </hardwareInterface>
-    </joint>
-    <actuator name="right_wheel_actuator">
-      <mechanicalReduction>1</mechanicalReduction>
-      <hardwareInterface>
-        VelocityJointInterface
-      </hardwareInterface>
-    </actuator>
-  </transmission>
-  <transmission name="left_wheel_transmission">
-    <type>transmission_interface/SimpleTransmission</type>
-    <joint name="joint_left_wheel">
-      <hardwareInterface>
-        hardware_interface/VelocityJointInterface
-      </hardwareInterface>
-    </joint>
-    <actuator name="left_wheel_actuator">
-      <mechanicalReduction>1</mechanicalReduction>
-      <hardwareInterface>
-        VelocityJointInterface
-      </hardwareInterface>
-    </actuator>
-  </transmission>
 </robot>

Commit message: Add lidar simulation

File: src/realsense_explorer_description/urdf/realsense_explorer.urdf (robot description, URDF)
Before this commit: robot realsense_explorer, 18 links, 17 joints
Links:
- added link lidar_link, mass 0.2; collision cylinder length=0.02 radius=0.04; visual cylinder length=0.02 radius=0.04
Joints:
- added joint lidar_joint: type fixed, parent robot_base, child lidar_link, origin xyz=0 0 0.132 rpy=0 0 0

File: src/realsense_explorer_description/urdf/realsense_explorer.urdf.xacro (robot description, xacro)
@@ -38,4 +38,36 @@
     </plugin>
   </gazebo>
+  <!--#####################  LIDAR ##########################-->
+  <gazebo reference="lidar_link">
+    <sensor name="lidar_rays" type="ray">
+      <pose>0 0 0 0 0 0</pose>
+      <visualize>False</visualize>
+      <update_rate>5</update_rate>
+      <ray>
+        <scan>
+          <horizontal>
+            <samples>719</samples>
+            <resolution>1</resolution>
+            <min_angle>-3.14159</min_angle>
+            <max_angle>3.14159</max_angle>
+          </horizontal>
+        </scan>
+        <range>
+          <min>0.05</min>
+          <max>20.0</max>
+          <resolution>0.01</resolution>
+        </range>
+        <noise>
+          <type>gaussian</type>
+          <mean>0.0</mean>
+          <stddev>0.005</stddev>
+        </noise>
+      </ray>
+      <plugin filename="libgazebo_ros_laser.so" name="gazebo_ros_head_hokuyo_controller">
+        <topicName>scan</topicName>
+        <frameName>lidar_link</frameName>
+      </plugin>
+    </sensor>
+  </gazebo>
   <link name="base_footprint"/>
   <link name="robot_base">
@@ -210,3 +242,28 @@
     <parent link="robot_base"/>
   </joint>
+  <!-- LIDAR Link -->
+  <link name="lidar_link">
+    <visual>
+      <geometry>
+        <cylinder radius="0.04" length="0.02"/> <!-- Adjust size as needed -->
+      </geometry>
+      <material name="grey"/>
+    </visual>
+    <collision>
+      <geometry>
+        <cylinder radius="0.04" length="0.02"/>
+      </geometry>
+    </collision>
+    <inertial>
+      <mass value="0.2"/>
+      <origin xyz="0 0 0"/>
+      <inertia ixx="8.67e-5" ixy="0.0" ixz="0.0" iyy="8.67e-5" iyz="0.0" izz="1.6e-4"/>
+    </inertial>
+  </link>
+  <!-- LIDAR Joint -->
+  <joint name="lidar_joint" type="fixed">
+    <parent link="robot_base"/>
+    <child link="lidar_link"/>
+    <origin xyz="0 0 0.132" rpy="0 0 0"/>
+  </joint>
 </robot>

Commit message: Build lidar model according to real robot

File: src/realsense_explorer_description/urdf/realsense_explorer.urdf (robot description, URDF)
Before this commit: robot realsense_explorer, 19 links, 18 joints
Links:
- added link lidar_bottom_link, mass 0.2; collision box size=0.05 0.052 0.03; visual box size=0.05 0.052 0.03
- added link lidar_connection_link, mass 0.2; collision box size=0.06 0.1 0.04; visual box size=0.06 0.1 0.04
- link lidar_link: geometry collision cylinder length=0.03 radius=0.02; visual cylinder length=0.03 radius=0.02
Joints:
- added joint lidar_bottom_joint: type fixed, parent robot_base, child lidar_bottom_link, origin xyz=0.025 0 0.175 rpy=0 0 0
- added joint lidar_connection_joint: type fixed, parent robot_base, child lidar_connection_link, origin xyz=0.02 0 0.144 rpy=0 0 0
- joint camera_joint: origin xyz=0.08 0 0.09 rpy=0 0 0 -> xyz=0.038 0 0.09 rpy=0 0 0
- joint lidar_joint: origin xyz=0 0 0.132 rpy=0 0 0 -> xyz=0.03 0 0.205 rpy=0 0 0

File: src/realsense_explorer_description/urdf/realsense_explorer.urdf.xacro (robot description, xacro)
@@ -4,5 +4,5 @@
   <link name="base_link" />
   <xacro:sensor_d435 name="camera" topics_ns="camera" parent="robot_base" publish_pointcloud="true" color_ur="20.0" ir_ur="20.0" depth_ur="20.0">
-    <origin xyz="0.08 0 0.09" rpy="0 0 0" />
+    <origin xyz="0.038 0 0.09" rpy="0 0 0" />
   </xacro:sensor_d435>
   <material name="invisible">
@@ -26,7 +26,7 @@
       <wheelDiameter>0.2</wheelDiameter>
       <robotBaseFrame>base_footprint</robotBaseFrame>
-      <torque>20</torque>
-      <maxVelocity>2.0</maxVelocity>
-      <maxAcceleration>3.0</maxAcceleration>
+      <torque>10</torque>
+      <maxVelocity>1</maxVelocity>
+      <maxAcceleration>2.0</maxAcceleration>
       <topicName>cmd_vel</topicName>
       <odometryTopic>odom</odometryTopic>
@@ -246,5 +246,5 @@
     <visual>
       <geometry>
-        <cylinder radius="0.04" length="0.02"/> <!-- Adjust size as needed -->
+        <cylinder radius="0.02" length="0.03"/> <!-- Adjust size as needed -->
       </geometry>
       <material name="grey"/>
@@ -252,5 +252,41 @@
     <collision>
       <geometry>
-        <cylinder radius="0.04" length="0.02"/>
+        <cylinder radius="0.02" length="0.03"/>
+      </geometry>
+    </collision>
+    <inertial>
+      <mass value="0.2"/>
+      <origin xyz="0 0 0"/>
+      <inertia ixx="8.67e-5" ixy="0.0" ixz="0.0" iyy="8.67e-5" iyz="0.0" izz="1.6e-4"/>
+    </inertial>
+  </link>
+  <link name="lidar_bottom_link">
+    <visual>
+      <geometry>
+        <box size="0.05 0.052 0.03"/> <!-- Adjust size as needed -->
+      </geometry>
+      <material name="grey"/>
+    </visual>
+    <collision>
+      <geometry>
+        <box size="0.05 0.052 0.03"/>
+      </geometry>
+    </collision>
+    <inertial>
+      <mass value="0.2"/>
+      <origin xyz="0 0 0"/>
+      <inertia ixx="8.67e-5" ixy="0.0" ixz="0.0" iyy="8.67e-5" iyz="0.0" izz="1.6e-4"/>
+    </inertial>
+  </link>
+  <link name="lidar_connection_link">
+    <visual>
+      <geometry>
+        <box size="0.06 0.1 0.04"/>
+      </geometry>
+      <material name="grey"/>
+    </visual>
+    <collision>
+      <geometry>
+        <box size="0.06 0.1 0.04"/>
       </geometry>
     </collision>
@@ -265,5 +301,15 @@
     <parent link="robot_base"/>
     <child link="lidar_link"/>
-    <origin xyz="0 0 0.132" rpy="0 0 0"/>
+    <origin xyz="0.03 0 0.205" rpy="0 0 0"/>
+  </joint>
+  <joint name="lidar_bottom_joint" type="fixed">
+    <parent link="robot_base"/>
+    <child link="lidar_bottom_link"/>
+    <origin xyz="0.025 0 0.175" rpy="0 0 0"/>
+  </joint>
+  <joint name="lidar_connection_joint" type="fixed">
+    <parent link="robot_base"/>
+    <child link="lidar_connection_link"/>
+    <origin xyz="0.02 0 0.144" rpy="0 0 0"/>
   </joint>
 </robot>
